Commit message: Updated passive view cam

File: URDF_files/L515_cam_with_stand.urdf (robot description, URDF)
Before this commit: robot D405_camera_with_stand, 3 links, 2 joints
Links:
- link horizontal_link: geometry visual box size=0.1 0.01 0.01
- link vertical_link: geometry visual box size=0.01 0.01 0.8
Joints:
- joint camera_joint: origin xyz=-0.25 0 -0.014 rpy=3.1416 0.7854 0 -> xyz=-0.05 0 -0.014 rpy=3.1416 0.5236 0
- joint vertical_to_horizontal: origin xyz=-0.245 0 1.005 -> xyz=-0.045 0 0.405

Commit message: Increase height of both cam

File: URDF_files/L515_cam_with_stand.urdf (robot description, URDF)
Before this commit: robot L515_camera_with_stand, 3 links, 2 joints
Joints:
- joint vertical_to_horizontal: origin xyz=-0.045 0 0.405 -> xyz=-0.045 0 0.75

Commit message: Change sim setup for real-world tests

File: URDF_files/L515_cam_with_stand.urdf (robot description, URDF)
Before this commit: robot L515_camera_with_stand, 3 links, 2 joints
Links:
- link vertical_link: geometry visual box size=0.01 0.01 0.5
Joints:
- joint vertical_to_horizontal: origin xyz=-0.045 0 0.405 -> xyz=-0.045 0 0.4

File: URDF_files/panda_modified.urdf (robot description, URDF)
Before this commit: robot panda, 15 links, 14 joints
Joints:
- joint camera_joint: origin xyz=0.035 0 -0.05 rpy=3.1416 0 1.5708  -> xyz=0.06 0 -0.06 rpy=3.1416 0 1.5708 

Commit message: Revert "Change sim setup for real-world tests"
This reverts commit dd50f6cb60a84cd6d0770305ffb076f56c476ed1.

File: URDF_files/L515_cam_with_stand.urdf (robot description, URDF)
Before this commit: robot L515_camera_with_stand, 3 links, 2 joints
Links:
- link vertical_link: geometry visual box size=0.01 0.01 0.8
Joints:
- joint vertical_to_horizontal: origin xyz=-0.045 0 0.4 -> xyz=-0.045 0 0.405

File: URDF_files/panda_modified.urdf (robot description, URDF)
Before this commit: robot panda, 15 links, 14 joints
Joints:
- joint camera_joint: origin xyz=0.06 0 -0.06 rpy=3.1416 0 1.5708  -> xyz=0.035 0 -0.05 rpy=3.1416 0 1.5708 
