Commit message: Correct panda_modified (img was flipped on y axis)

File: URDF_files/panda_modified.urdf (robot description, URDF)
Before this commit: robot panda, 14 links, 13 joints
Joints:
- joint camera_joint: origin xyz=0.035 0 -0.05 rpy=0 -3.1416 0 -> xyz=0.035 0 -0.05 rpy=3.1416 0 1.5708 

Commit message: Revert "Correct panda_modified (img was flipped on y axis)"
This reverts commit d271fc1d1b18c32136295f6c5072fa76620890ea.

File: URDF_files/panda_modified.urdf (robot description, URDF)
Before this commit: robot panda, 14 links, 13 joints
Joints:
- joint camera_joint: origin xyz=0.035 0 -0.05 rpy=3.1416 0 1.5708  -> xyz=0.035 0 -0.05 rpy=0 -3.1416 0

Commit message: Fixed robot-cam rendering

File: URDF_files/panda_modified.urdf (robot description, URDF)
Before this commit: robot panda, 14 links, 13 joints
Links:
- added link thin_link, mass 0.0; visual box size=0.0001 0.0001 0.0001
Joints:
- added joint fixed_joint: type fixed, parent camera_link, child thin_link, origin xyz=0 0 -0.023 rpy=0 0 0

Commit message: Active-cam can now see gripper

File: URDF_files/panda_modified.urdf (robot description, URDF)
Before this commit: robot panda, 15 links, 14 joints
Joints:
- joint camera_joint: origin xyz=0.035 0 -0.05 rpy=3.1416 0 1.5708  -> xyz=0.035 0 -0.09 rpy=3.1416 0 1.5708 

Commit message: Change active cam to not see gripper for reach and push tasks

File: URDF_files/panda_modified.urdf (robot description, URDF)
Before this commit: robot panda, 15 links, 14 joints
Joints:
- joint camera_joint: origin xyz=0.035 0 -0.09 rpy=3.1416 0 1.5708  -> xyz=0.035 0 -0.05 rpy=3.1416 0 1.5708 

Commit message: Try black table

File: URDF_files/panda_modified.urdf (robot description, URDF)
Before this commit: robot panda, 15 links, 14 joints
Joints:
- joint camera_joint: origin xyz=0.035 0 -0.05 rpy=3.1416 0 1.5708  -> xyz=0.065 0 -0.05 rpy=3.1416 0 1.5708 

Commit message: Increase camera away further

File: URDF_files/panda_modified.urdf (robot description, URDF)
Before this commit: robot panda, 15 links, 14 joints
Joints:
- joint camera_joint: origin xyz=0.065 0 -0.05 rpy=3.1416 0 1.5708  -> xyz=0.085 0 -0.05 rpy=3.1416 0 1.5708 

Commit message: Minor changes

File: URDF_files/panda_modified.urdf (robot description, URDF)
Before this commit: robot panda, 15 links, 14 joints
Joints:
- joint camera_joint: origin xyz=0.035 0 -0.05 rpy=3.1416 0 1.5708  -> xyz=0.085 0 -0.05 rpy=3.1416 0 1.5708 

Commit message: Revert "Merge branch 'philip4_dual_deep_reachandpush_joints' of github.com:NUSLCC/panda_gym_cam into philip4_dual_deep_reachandpush_joints"
This reverts commit 6c2a4de39056e701969172924e13046638f1a470, reversing
changes made to b35c21409966bd3509e7b03b7c63b9c34edafa81.

File: URDF_files/panda_modified.urdf (robot description, URDF)
Before this commit: robot panda, 15 links, 14 joints
Joints:
- joint camera_joint: origin xyz=0.085 0 -0.05 rpy=3.1416 0 1.5708  -> xyz=0.035 0 -0.05 rpy=3.1416 0 1.5708 

Commit message: Changes for push cam real

File: URDF_files/panda_modified.urdf (robot description, URDF)
Before this commit: robot panda, 15 links, 14 joints
Joints:
- joint camera_joint: origin xyz=0.085 0 -0.05 rpy=3.1416 0 1.5708  -> xyz=0.065 0 -0.05 rpy=3.1416 0 1.5708 
